Commit message: update

File: urdf/robot1.xacro (robot description, xacro)
@@ -13,6 +13,6 @@
 		<geometry>
        			<cylinder length="${length_wheel}" radius="${radius_wheel}"/>
-     	</geometry>
-	</xacro:macro>
+     		</geometry>
+    </xacro:macro>
 	  <link name="link_chassis">
     <!-- pose and inertial -->

File: urdf/robot1_arm.urdf (robot description, URDF)
Before this commit: robot Robot1, 3 links, 2 joints
Links:
- added link arm_1; visual box size=0.05 .05 0.5
- added link arm_2; visual box size=0.05 0.05 0.5
- added link arm_base; visual box size=0.1 .1 .1
Joints:
- added joint arm_1_to_arm_base: type revolute, parent arm_base, child arm_1, origin xyz=0 0 0.15, axis 1 0 0, limit lower=-1.0 upper=1.0 effort=100.0 velocity=0.5
- added joint arm_2_to_arm_1: type revolute, parent arm_1, child arm_2, origin xyz=0.0 0 0.45, axis 1 0 0, limit lower=-2.5 upper=2.5 effort=100.0 velocity=0.5
- added joint base_to_arm_base: type continuous, parent link_chassis, child arm_base, origin xyz=0 0 0, axis 0 0 1
